File: PCB/odyssey67.kicad_pcb (KiCad board)
At the start: 2 copper layers, 312.7 x 103.2 mm, 137 parts, among them U1 Elite-C

Commit message: Updated PCB
Parts:
- added REF**: OSHW-Logo_11.4x12mm_SilkScreen, Symbol:OSHW-Logo_11.4x12mm_SilkScreen, B.Cu at (218.3, 184.9)
- added REF**: OSHW-Logo_11.4x12mm_SilkScreen, Symbol:OSHW-Logo_11.4x12mm_SilkScreen, F.Cu at (218.3, 184.9)
- moved D14 7.94 mm to (306.4, 111.9)
- moved D15 2.38 mm to (339.7, 111.9)
- moved D43 1.59 mm to (337.3, 150.0)
- moved D13 0.79 mm to (303.2, 111.9)
Routing:
- net Net-(D14-Pad2): track 11.9 -> 19.8 mm
- net Net-(D15-Pad2): track 17.4 -> 15.0 mm
- net Net-(D43-Pad2): track 13.1 -> 14.7 mm
- net R0: track 272.0 -> 272.9 mm
- net Net-(D13-Pad2): track 7.58 -> 6.78 mm
Other:
- board text added: "Rev 2.1 08/2020"
- board text added: "Somewhere, something incredible is waiting to be known."
- board text removed: "Rev 1.0 04/2020"

Commit message: Update PCB / Plates
Parts:
- removed REF** (x2): OSHW-Logo_11.4x12mm_SilkScreen, Symbol:OSHW-Logo_11.4x12mm_SilkScreen
